File: ffc-breakout_v1.sch (EAGLE design)
At the start: 5 parts, among them X2 AMP_SFW16R-2STE1LF

Commit message: BOM  + minor FFC update
Parts:
- X1: device pinhead:PINHD-2X8/90 -> pinhead:PINHD-2X8
Changed lines of the file:
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@@
 <parts>
 <part name="X2" library="components" deviceset="AMP_SFW16R-2STE1LF" device=""/>
-<part name="X1" library="pinhead" library_urn="urn:adsk.eagle:library:325" deviceset="PINHD-2X8" device="/90" package3d_urn="urn:adsk.eagle:package:22488/1"/>
+<part name="X1" library="pinhead" library_urn="urn:adsk.eagle:library:325" deviceset="PINHD-2X8" device="" package3d_urn="urn:adsk.eagle:package:22481/2"/>
 <part name="X3" library="pinhead" library_urn="urn:adsk.eagle:library:325" deviceset="PINHD-1X3" device="/90" package3d_urn="urn:adsk.eagle:package:22459/1"/>
 <part name="SJ1" library="jumper" library_urn="urn:adsk.eagle:library:252" deviceset="SJ2W" device="" package3d_urn="urn:adsk.eagle:package:15474/1"/>
